File: e-ink-frdm-adapter.kicad_pcb (KiCad board)
At the start: 2 copper layers, 30.5 x 28.6 mm, 23 parts, among them P1 2-1734839-4, P2 68000-110HLF, Q1 MF-DSC-SOT233-BSS138

Commit message: Use bottom contact FPC conn footprint
Parts:
- P1: footprint muchi_footprints:TE-2-1734839-4 -> muchi_footprints:TE-2-1734592-4-bottom_contact
Changed lines of the file:
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@@
     )
   )
-  (module muchi_footprints:TE-2-1734839-4 locked (layer F.Cu)
+  (module Resistors_SMD:R_0402 placed (layer F.Cu)
+    (at 115.57 72.39 180)
+    (descr "Resistor SMD 0402, reflow soldering, Vishay (see dcrcw.pdf)")
+    (tags "resistor 0402")
+    (attr smd)
+    (fp_text reference C13 (at 0 -1.8 180) (layer F.SilkS)
+      (effects (font (size 1 1) (thickness 0.15)))
+    )
+    (fp_text value MF-CAP-0402-1uF (at 0 1.8 180) (layer F.Fab)
+      (effects (font (size 1 1) (thickness 0.15)))
+    )
+    (fp_line (start -0.95 -0.65) (end 0.95 -0.65) (layer F.CrtYd) (width 0.05))
+    (fp_line (start -0.95 0.65) (end 0.95 0.65) (layer F.CrtYd) (width 0.05))
+    (fp_line (start -0.95 -0.65) (end -0.95 0.65) (layer F.CrtYd) (width 0.05))
+    (fp_line (start 0.95 -0.65) (end 0.95 0.65) (layer F.CrtYd) (width 0.05))
+    (fp_line (start 0.25 -0.525) (end -0.25 -0.525) (layer F.SilkS) (width 0.15))
+    (fp_line (start -0.25 0.525) (end 0.25 0.525) (layer F.SilkS) (width 0.15))
+    (pad 1 smd rect (at -0.45 0 180) (size 0.4 0.6) (layers F.Cu F.Paste F.Mask)
+      (net 13 /V3.3))
+    (pad 2 smd rect (at 0.45 0 180) (size 0.4 0.6) (layers F.Cu F.Paste F.Mask)
+      (net 3 GND))
+    (model Resistors_SMD.3dshapes/R_0402.wrl
+      (at (xyz 0 0 0))
+      (scale (xyz 1 1 1))
+      (rotate (xyz 0 0 0))
+    )
+  )
+  (module Resistors_SMD:R_0402 placed (layer F.Cu)
+    (at 115.57 71.12 180)
+    (descr "Resistor SMD 0402, reflow soldering, Vishay (see dcrcw.pdf)")
+    (tags "resistor 0402")
+    (attr smd)
+    (fp_text reference C12 (at 0.254 1.651 180) (layer F.SilkS)
+      (effects (font (size 1 1) (thickness 0.15)))
+    )
+    (fp_text value MF-CAP-0402-1uF (at 0 1.8 180) (layer F.Fab)
+      (effects (font (size 1 1) (thickness 0.15)))
+    )
+    (fp_line (start -0.95 -0.65) (end 0.95 -0.65) (layer F.CrtYd) (width 0.05))
+    (fp_line (start -0.95 0.65) (end 0.95 0.65) (layer F.CrtYd) (width 0.05))
+    (fp_line (start -0.95 -0.65) (end -0.95 0.65) (layer F.CrtYd) (width 0.05))
+    (fp_line (start 0.95 -0.65) (end 0.95 0.65) (layer F.CrtYd) (width 0.05))
+    (fp_line (start 0.25 -0.525) (end -0.25 -0.525) (layer F.SilkS) (width 0.15))
+    (fp_line (start -0.25 0.525) (end 0.25 0.525) (layer F.SilkS) (width 0.15))
+    (pad 1 smd rect (at -0.45 0 180) (size 0.4 0.6) (layers F.Cu F.Paste F.Mask)
+      (net 13 /V3.3))
+    (pad 2 smd rect (at 0.45 0 180) (size 0.4 0.6) (layers F.Cu F.Paste F.Mask)
+      (net 3 GND))
+    (model Resistors_SMD.3dshapes/R_0402.wrl
+      (at (xyz 0 0 0))
+      (scale (xyz 1 1 1))
+      (rotate (xyz 0 0 0))
+    )
+  )
+  (module muchi_footprints:TE-2-1734592-4-bottom_contact locked (layer F.Cu)
     (at 121.92 53.34 180)
-    (fp_text reference P1 (at -13.335 -22.225 180) (layer F.SilkS)
+    (fp_text reference P1 (at 0.5 -6.5 180) (layer F.SilkS)
       (effects (font (size 1.5 1.5) (thickness 0.15)))
     )
@@
     (pad "" smd rect (at 7.5 -0.5 180) (size 2.3 3.1) (layers F.Cu F.Paste F.Mask))
   )
-  (module Resistors_SMD:R_0402 placed (layer F.Cu)
-    (at 115.57 72.39 180)
-    (descr "Resistor SMD 0402, reflow soldering, Vishay (see dcrcw.pdf)")
-    (tags "resistor 0402")
-    (attr smd)
-    (fp_text reference C13 (at 0 -1.8 180) (layer F.SilkS)
-      (effects (font (size 1 1) (thickness 0.15)))
-    )
-    (fp_text value MF-CAP-0402-1uF (at 0 1.8 180) (layer F.Fab)
-      (effects (font (size 1 1) (thickness 0.15)))
-    )
-    (fp_line (start -0.95 -0.65) (end 0.95 -0.65) (layer F.CrtYd) (width 0.05))
-    (fp_line (start -0.95 0.65) (end 0.95 0.65) (layer F.CrtYd) (width 0.05))
-    (fp_line (start -0.95 -0.65) (end -0.95 0.65) (layer F.CrtYd) (width 0.05))
-    (fp_line (start 0.95 -0.65) (end 0.95 0.65) (layer F.CrtYd) (width 0.05))
-    (fp_line (start 0.25 -0.525) (end -0.25 -0.525) (layer F.SilkS) (width 0.15))
-    (fp_line (start -0.25 0.525) (end 0.25 0.525) (layer F.SilkS) (width 0.15))
-    (pad 1 smd rect (at -0.45 0 180) (size 0.4 0.6) (layers F.Cu F.Paste F.Mask)
-      (net 13 /V3.3))
-    (pad 2 smd rect (at 0.45 0 180) (size 0.4 0.6) (layers F.Cu F.Paste F.Mask)
-      (net 3 GND))
-    (model Resistors_SMD.3dshapes/R_0402.wrl
-      (at (xyz 0 0 0))
-      (scale (xyz 1 1 1))
-      (rotate (xyz 0 0 0))
-    )
-  )
-  (module Resistors_SMD:R_0402 placed (layer F.Cu)
-    (at 115.57 71.12 180)
-    (descr "Resistor SMD 0402, reflow soldering, Vishay (see dcrcw.pdf)")
-    (tags "resistor 0402")
-    (attr smd)
-    (fp_text reference C12 (at 0.254 1.651 180) (layer F.SilkS)
-      (effects (font (size 1 1) (thickness 0.15)))
-    )
-    (fp_text value MF-CAP-0402-1uF (at 0 1.8 180) (layer F.Fab)
-      (effects (font (size 1 1) (thickness 0.15)))
-    )
-    (fp_line (start -0.95 -0.65) (end 0.95 -0.65) (layer F.CrtYd) (width 0.05))
-    (fp_line (start -0.95 0.65) (end 0.95 0.65) (layer F.CrtYd) (width 0.05))
-    (fp_line (start -0.95 -0.65) (end -0.95 0.65) (layer F.CrtYd) (width 0.05))
-    (fp_line (start 0.95 -0.65) (end 0.95 0.65) (layer F.CrtYd) (width 0.05))
-    (fp_line (start 0.25 -0.525) (end -0.25 -0.525) (layer F.SilkS) (width 0.15))
-    (fp_line (start -0.25 0.525) (end 0.25 0.525) (layer F.SilkS) (width 0.15))
-    (pad 1 smd rect (at -0.45 0 180) (size 0.4 0.6) (layers F.Cu F.Paste F.Mask)
-      (net 13 /V3.3))
-    (pad 2 smd rect (at 0.45 0 180) (size 0.4 0.6) (layers F.Cu F.Paste F.Mask)
-      (net 3 GND))
-    (model Resistors_SMD.3dshapes/R_0402.wrl
-      (at (xyz 0 0 0))
-      (scale (xyz 1 1 1))
-      (rotate (xyz 0 0 0))
-    )
-  )
   (gr_text "Muchi Corporation\ne-ink display adapter board\nv0.1" (at 135.001 58.547 270) (layer F.SilkS)

Commit message: Regenerate with latest changes
Other:
- board text added: "Muchi Corporation e-ink display adapter board v0.2"
- board text removed: "Muchi Corporation e-ink display adapter board v0.1"
Changed lines of the file:
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@@
     (area 102.215477 50.904999 137.235001 89.55)
     (thickness 1.6)
-    (drawings 7)
+    (drawings 8)
     (tracks 231)
     (zones 0)
@@
     (pad "" smd rect (at 7.5 -0.5 180) (size 2.3 3.1) (layers F.Cu F.Paste F.Mask))
   )
-  (gr_text "Muchi Corporation\ne-ink display adapter board\nv0.1" (at 135.001 58.547 270) (layer F.SilkS)
+  (gr_circle (center 132.588 54.229) (end 132.461 53.721) (layer F.SilkS) (width 1))
+  (gr_text "Muchi Corporation\ne-ink display adapter board\nv0.2" (at 135.001 58.547 270) (layer F.SilkS)
     (effects (font (size 0.5 0.5) (thickness 0.125)))
   )
